File: pcbs/eggada50_wireless_manually_routed.kicad_pcb (KiCad board)
At the start: 2 copper layers, 140.4 x 102.8 mm, 114 parts

Commit message: updates on right angled traces
Routing:
- net R0: track 276.2 -> 279.1 mm
Changed lines of the file:
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@@
-	)
-	(segment
-		(start 220.403 72.150364)
-		(end 220.403 62.401)
-		(width 0.2)
-		(layer "F.Cu")
-		(net 34)
 	)
 	(segment
@@
 	)
 	(segment
-		(start 224.25 109.69)
-		(end 224.25 74.4)
+		(start 94.865 102.59)
+		(end 110.49 102.59)
 		(width 0.2)
 		(layer "F.Cu")
@@
 	)
 	(segment
-		(start 94.865 102.59)
-		(end 110.49 102.59)
+		(start 220.403 62.401)
+		(end 220.403 72.150364)
 		(width 0.2)
 		(layer "F.Cu")
@@
 	)
 	(segment
+		(start 226.63 79.03)
+		(end 224.25 81.41)
+		(width 0.2)
+		(layer "F.Cu")
+		(net 34)
+	)
+	(segment
+		(start 221.772636 73.52)
+		(end 224.93 73.52)
+		(width 0.2)
+		(layer "F.Cu")
+		(net 34)
+	)
+	(segment
+		(start 221.104 61.7)
+		(end 220.403 62.401)
+		(width 0.2)
+		(layer "F.Cu")
+		(net 34)
+	)
+	(segment
 		(start 217.77 120.47)
 		(end 221.95 116.29)
@@
 	)
 	(segment
-		(start 224.25 74.4)
-		(end 222.652636 74.4)
+		(start 224.93 73.52)
+		(end 226.63 75.22)
+		(width 0.2)
+		(layer "F.Cu")
+		(net 34)
+	)
+	(segment
+		(start 224.25 81.41)
+		(end 224.25 109.69)
+		(width 0.2)
+		(layer "F.Cu")
+		(net 34)
+	)
+	(segment
+		(start 220.403 72.150364)
+		(end 221.772636 73.52)
 		(width 0.2)
 		(layer "F.Cu")
@@
 		(start 210.885941 124.811088)
 		(end 213.428912 124.811088)
-		(width 0.2)
-		(layer "F.Cu")
-		(net 34)
-	)
-	(segment
-		(start 222.652636 74.4)
-		(end 220.403 72.150364)
 		(width 0.2)
 		(layer "F.Cu")
@@
 	)
 	(segment
+		(start 226.63 75.22)
+		(end 226.63 79.03)
+		(width 0.2)
+		(layer "F.Cu")
+		(net 34)
+	)
+	(segment
 		(start 222.284 61.7)
 		(end 221.104 61.7)
@@
 		(width 0.2)
 		(layer "F.Cu")
-		(net 34)
-	)
-	(segment
-		(start 220.403 62.401)
-		(end 221.104 61.7)
-		(width 0.2)
-		(layer "F.Cu")
